File: public/ParametricPCB/03-compactAudioMotionSquarePCB/03_compactSquareLedHapticPCB.kicad_pcb (KiCad board)
At the start: 2 copper layers, 38 x 38 mm, 29 parts

Commit message: ImprovementsPCBgenerator
Parts:
- ? (x4): footprint tscircuit:platedhole_circle_holeDiameter3.2mm_outerDiameter6mm -> tscircuit:platedhole_circle_holeDiameter3.2mm_outerDiameter4.8mm
- moved C_VIN 0.30 mm to (92.5, 82.9)
Routing:
- net Q_LED_PWR____pin3_to__J_LED____pin1: track 73.8 -> 111.2 mm, vias 8 -> 4
- net U_MCU____pin11_to__Q_FET____pin1: track 50.6 -> 74.2 mm, vias 1 -> 4
- net U_MCU____pin1_to__U_CHG____pin4: track 38.1 -> 51.4 mm, vias 2 -> 4
- net D_HAP____pin1_to__J_HAP_L____pin1: track 64.6 -> 71.8 mm, vias 5 -> 4
- net U_MCU____pin6_to__U_IMU____pin4: track 23.2 -> 29.1 mm
- net Q_FET____pin3_to__J_HAP_L____pin2: track 44.5 -> 40.9 mm, vias 8 -> 2
- net U_MCU____pin16_to__J_LED3____pin2: track 29.2 -> 32.3 mm, vias 5 -> 2
- net U_MCU____pin4_to__J_MIC_MAX____pin3: track 21.2 -> 24.0 mm, vias 2 -> 1
- net Q_LED_EN____pin3_to__Q_LED_PWR____pin1: track 12.9 -> 10.2 mm
- net SW_EXT____pin2_to__Q_PWR____pin3: track 32.8 -> 34.5 mm, vias 4 -> 3
- net U_MCU____pin3_to__U_IMU____pin1: track 70.4 -> 68.8 mm, vias 7 -> 9
- net U_MCU____pin5_to__J_MIC_INMP____pin2: track 26.6 -> 25.0 mm
- net U_MCU____pin14_to__Q_LED_EN____pin1: track 13.0 -> 14.4 mm, vias 2 -> 1
- net C_VIN____pin2_to__U_CHG____pin2: track 70.1 -> 69.1 mm, vias 8 -> 9
- net U_MCU____pin10_to__J_LED____pin2: track 10.3 -> 11.2 mm
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