File: public/ParametricPCB/03-compactAudioMotionSquarePCB/gerber_export/03_compactSquareLedHapticPCB.kicad_pcb (KiCad board)
At the start: 2 copper layers, 38 x 38 mm, 29 parts

Commit message: ImprovementsPCBgenerator
Parts:
- ? (x4): footprint tscircuit:platedhole_circle_holeDiameter3.2mm_outerDiameter6mm -> tscircuit:platedhole_circle_holeDiameter3.2mm_outerDiameter4.8mm
- moved C_VIN 0.30 mm to (92.5, 82.9)
Routing:
- net Q_LED_PWR____pin3_to__J_LED____pin1: track 76.9 -> 111.2 mm, vias 10 -> 4
- net U_MCU____pin11_to__Q_FET____pin1: track 44.4 -> 74.2 mm, vias 3 -> 4
- net U_CHG____pin3_to__C_BAT____pin1: track 72.0 -> 59.6 mm, vias 5 -> 7
- net U_MCU____pin2_to__U_IMU____pin2: track 93.3 -> 81.1 mm, vias 8 -> 6
- net U_MCU____pin15_to__J_LED2____pin2: track 25.7 -> 16.8 mm, vias 2 -> 1
- net D_HAP____pin1_to__J_HAP_L____pin1: track 63.4 -> 71.8 mm, vias 2 -> 4
- net U_MCU____pin7_to__U_IMU____pin3: track 33.6 -> 25.4 mm, vias 3 -> 1
- net C_VIN____pin2_to__U_CHG____pin2: track 62.7 -> 69.1 mm, vias 1 -> 9
- net U_MCU____pin1_to__U_CHG____pin4: track 45.6 -> 51.4 mm, vias 0 -> 4
- net Q_FET____pin3_to__J_HAP_L____pin2: track 46.5 -> 40.9 mm, vias 4 -> 2
- net Q_LED_EN____pin3_to__Q_LED_PWR____pin1: track 13.9 -> 10.2 mm, vias 2 -> 0
- net SW_EXT____pin2_to__Q_PWR____pin3: track 31.3 -> 34.5 mm, vias 2 -> 3
- net U_MCU____pin12_to__J_MIC_INMP____pin4: track 14.9 -> 17.5 mm
- net U_MCU____pin3_to__U_IMU____pin1: track 66.9 -> 68.8 mm, vias 2 -> 9
- net U_CHG____pin5_to__R_PROG____pin1: track 4.65 -> 3.09 mm, vias 2 -> 0
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